File: Hardware/SumoRc/Sumorc.kicad_sch (KiCad schematic)
At the start: 8 parts, among them SW1 SW_SPDT, U1 ESP32_DevKit_V1_DOIT, U2 Mini360

Commit message: se actualizo el esquematico y pcb
Parts:
- removed BTS7960_1, BTS7960_2: Conn_01x05, Connector_JST:JST_EH_B5B-EH-A_1x05_P2.50mm_Vertical, symbol Connector_Generic:Conn_01x05
- removed U2: Mini360, Mini360_step-down:Mini360_step-down, symbol mini360:Mini360
- added J1: BTS7960_1, EESTN5:JST-4V, symbol EESTN5:Screw_Terminal_01x04
- added J2: BTS7960_2, EESTN5:JST-4V, symbol EESTN5:Screw_Terminal_01x04
- added U2: LF15_TO220, EESTN5:to220, symbol Regulator_Linear:LF15_TO220
Connections:
- net GND: now also J1.4 (Pin_4), J2.1 (Pin_1), U2.2 (GND)
- net LPWM_1: now also J1.1 (Pin_1)
- net LPWM_2: now also J2.3 (Pin_3)
- net RPWM_1: now also J1.2 (Pin_2)
- net RPWM_2: now also J2.4 (Pin_4)
- net +5V: now reaches U1.18 (VIN)
- net +5V: now also C1.1, C2.1, J1.3 (Pin_3), J2.2 (Pin_2), U2.3 (VO)
- net at SW1.1 (A): now also U2.1 (VI)
- removed net +3V3: C1.1, C2.1, U1.19 (3V3)
- net EN_1: no longer names the net of U1.10 (IO27)
Other:
- moved on the sheet: C1, C2, Logica_7.4v1, SW1

Commit message: update
Parts:
- U2: footprint EESTN5:to220 -> EESTN5:TO-220
Changed lines of the file:
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@@
 			)
 		)
-		(property "Footprint" "EESTN5:to220"
+		(property "Footprint" "EESTN5:TO-220"
 			(at 77.47 29.845 0)
 			(effects

Commit message: update Hardware
Parts:
- C2: footprint Capacitor_THT:C_Disc_D5.0mm_W2.5mm_P5.00mm -> Capacitor_SMD:C_0805_2012Metric_Pad1.18x1.45mm_HandSolder
- J1, J2: footprint EESTN5:JST-4V -> Connector_JST:JST_EH_B4B-EH-A_1x04_P2.50mm_Vertical
- U2: footprint EESTN5:TO-220 -> Package_TO_SOT_SMD:TO-263-3_TabPin2
Changed lines of the file:
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@@
 			)
 		)
-		(property "Footprint" "Capacitor_THT:C_Disc_D5.0mm_W2.5mm_P5.00mm"
+		(property "Footprint" "Capacitor_SMD:C_0805_2012Metric_Pad1.18x1.45mm_HandSolder"
 			(at 96.2152 43.18 0)
 			(effects
@@
 			)
 		)
-		(property "Footprint" "EESTN5:JST-4V"
+		(property "Footprint" "Connector_JST:JST_EH_B4B-EH-A_1x04_P2.50mm_Vertical"
 			(at 198.12 40.64 0)
 			(effects
@@
 			)
 		)
-		(property "Footprint" "EESTN5:TO-220"
+		(property "Footprint" "Package_TO_SOT_SMD:TO-263-3_TabPin2"
 			(at 77.47 29.845 0)
 			(effects
@@
 			)
 		)
-		(property "Footprint" "EESTN5:JST-4V"
+		(property "Footprint" "Connector_JST:JST_EH_B4B-EH-A_1x04_P2.50mm_Vertical"
 			(at 166.37 40.64 0)
 			(effects
