File: Hardware/SumoRc/Sumorc.kicad_pcb (KiCad board)
At the start: 2 copper layers, 8 parts, among them SW1 SW_SPDT, U1 ESP32_DevKit_V1_DOIT, U2 Mini360

Commit message: se actualizo el esquematico y pcb
Parts:
- removed BTS7960_1, BTS7960_2: Conn_01x05, Connector_JST:JST_EH_B5B-EH-A_1x05_P2.50mm_Vertical
- added J1: BTS7960_1, EESTN5:JST-4V, F.Cu at (155.2, 75.4)
- added J2: BTS7960_2, EESTN5:JST-4V, F.Cu at (155.1, 87.7)
- added REF**: MountingHole_2.1mm, MountingHole:MountingHole_2.1mm, F.Cu at (167.8, 48.4)
- added REF**: MountingHole_2.1mm, MountingHole:MountingHole_2.1mm, F.Cu at (167.8, 102.7)
- added REF**: MountingHole_2.1mm, MountingHole:MountingHole_2.1mm, F.Cu at (123.8, 48.4)
- added REF**: MountingHole_2.1mm, MountingHole:MountingHole_2.1mm, F.Cu at (123.8, 102.7)
- U2: value Mini360 -> LF15_TO220; footprint Mini360_step-down:Mini360_step-down -> EESTN5:to220
- moved U2 85.2 mm to (165.4, 63.9)
- moved SW1 84.7 mm to (165.3, 78.5)
- moved Logica_7.4v1 84.7 mm to (165.3, 93.7), turned to -90 degrees
- moved C1 77.1 mm to (155.8, 60.1), turned to -90 degrees
- moved C2 68.9 mm to (153.3, 54.6), turned to 0 degrees
- moved U1 34.3 mm to (136.3, 77.4)
Connections:
- C1 pad 1: +3V3 -> +5V
- C2 pad 1: +3V3 -> +5V
- U1 pad 10: EN_1 -> unconnected-(U1-IO27-Pad10)
- U1 pad 18: unconnected-(U1-VIN-Pad18) -> +5V
- U1 pad 19: +3V3 -> unconnected-(U1-3V3-Pad19)
- U2 pad 1: GND -> Net-(SW1-A)
- U2 pad 2: Net-(SW1-A) -> GND
- U2 pad 3: GND -> +5V
Routing:
- net +5V: track 0.00 -> 60.6 mm
- net Net-(SW1-B): track 0.00 -> 17.7 mm
- net RPWM_2: track 0.00 -> 6.98 mm
- net LPWM_1: track 0.00 -> 6.80 mm
- net LPWM_2: track 0.00 -> 6.78 mm
- net RPWM_1: track 0.00 -> 6.58 mm
- net Net-(SW1-A): track 0.00 -> 6.17 mm
- added copper zone on B.Cu, net GND
Other:
- board outline added: 50 x 60 mm

Commit message: update
Parts:
- U2: footprint EESTN5:to220 -> EESTN5:TO-220
- moved U2 8.44 mm to (166.0, 55.5)
- moved C1 7.85 mm to (159.0, 53.0), turned to 90 degrees
- moved SW1 5.89 mm to (166.0, 72.7)
- moved Logica_7.4v1 5.79 mm to (166.0, 87.9)
- moved C2 0.75 mm to (154.0, 54.5), turned to 90 degrees
Routing:
- net Net-(SW1-A): track 6.17 -> 9.96 mm
- net Net-(SW1-B): track 17.7 -> 19.1 mm

Commit message: update Hardware
Parts:
- C2: footprint Capacitor_THT:C_Disc_D5.0mm_W2.5mm_P5.00mm -> Capacitor_SMD:C_0805_2012Metric_Pad1.18x1.45mm_HandSolder; moved to B.Cu
- J1, J2: footprint EESTN5:JST-4V -> Connector_JST:JST_EH_B4B-EH-A_1x04_P2.50mm_Vertical
- U2: footprint EESTN5:TO-220 -> Package_TO_SOT_SMD:TO-263-3_TabPin2; moved to B.Cu
- moved C2 7.22 mm to (149.1, 49.2)
- moved C1 5.17 mm to (154.6, 50.3)
- moved J2 3.35 mm to (155.1, 91.0)
- moved U2 2.90 mm to (163.6, 57.1), turned to 0 degrees
Routing:
- net +5V: track 60.1 -> 14.1 mm
- net Net-(SW1-A): track 9.96 -> 16.2 mm
- net RPWM_1: track 6.58 -> 9.61 mm
- net LPWM_1: track 6.80 -> 9.16 mm

Commit message: se actualizo el PCB
Parts:
- moved Logica_7.4v1 1.96 mm to (164.0, 87.8)
- moved SW1 1.96 mm to (164.0, 72.7)
Routing:
- net Net-(SW1-A): track 16.2 -> 14.2 mm
- net Net-(SW1-B): track 19.1 -> 17.5 mm
- net LPWM_1: track 9.16 -> 10.0 mm
Changed lines of the file:
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@@
 	(footprint "RamLib:SW_SPDT_TH_Vertical"
 		(layer "F.Cu")
-		(at 166 72.7)
+		(at 164.04 72.65)
 		(descr "Switch inverseur")
 		(tags "SWITCH DEV")
@@
 	(footprint "XT30UPB-M:AMASS_XT30UPB-M"
 		(layer "F.Cu")
-		(at 166 87.9 -90)
+		(at 164.04 87.85 -90)
 		(property "Reference" "Logica_7.4v1"
 			(at -2.075 -3.675 90)
@@
 	)
 	(segment
-		(start 152.45 76.4)
-		(end 152.45 74)
-		(width 1)
-		(layer "B.Cu")
-		(net 2)
-	)
-	(segment
-		(start 151.41 77.44)
-		(end 152.45 76.4)
-		(width 1)
-		(layer "B.Cu")
-		(net 2)
-	)
-	(segment
-		(start 152.45 74)
-		(end 153.55026 72.89974)
-		(width 1)
-		(layer "B.Cu")
-		(net 2)
-	)
-	(segment
-		(start 153.55026 72.89974)
-		(end 155.15 72.89974)
-		(width 1)
-		(layer "B.Cu")
-		(net 2)
-	)
-	(segment
 		(start 149 77.44)
 		(end 151.41 77.44)
@@
 	)
 	(segment
-		(start 152.47 79.98)
-		(end 155.15 77.3)
+		(start 152.2 76.65)
+		(end 152.2 73.61)
 		(width 1)
 		(layer "B.Cu")
+		(net 2)
+	)
+	(segment
+		(start 151.41 77.44)
+		(end 152.2 76.65)
+		(width 1)
+		(layer "B.Cu")
+		(net 2)
+	)
+	(segment
+		(start 152.2 73.61)
+		(end 152.91026 72.89974)
+		(width 1)
+		(layer "B.Cu")
+		(net 2)
+	)
+	(segment
+		(start 152.91026 72.89974)
+		(end 155.15 72.89974)
+		(width 1)
+		(layer "B.Cu")
+		(net 2)
+	)
+	(segment
+		(start 153.93 79.98)
+		(end 155.15 78.76)
+		(width 1)
+		(layer "B.Cu")
 		(net 3)
 	)
 	(segment
-		(start 155.15 77.3)
+		(start 155.15 78.76)
 		(end 155.15 75.39974)
 		(width 1)
@@
 	(segment
 		(start 149 79.98)
-		(end 152.47 79.98)
+		(end 153.93 79.98)
 		(width 1)
 		(layer "B.Cu")
@@
 	)
 	(segment
-		(start 166 85.4)
-		(end 163.4 85.4)
-		(width 1.25)
+		(start 167.78 81.61)
+		(end 167.78 73.43)
+		(width 1)
 		(layer "B.Cu")
 		(net 9)
 	)
 	(segment
-		(start 162 74)
-		(end 163.3 72.7)
-		(width 1.25)
+		(start 167 72.65)
+		(end 164.04 72.65)
+		(width 1)
 		(layer "B.Cu")
 		(net 9)
 	)
 	(segment
-		(start 163.3 72.7)
-		(end 166 72.7)
-		(width 1.25)
+		(start 164.04 85.35)
+		(end 167.78 81.61)
+		(width 1)
 		(layer "B.Cu")
 		(net 9)
 	)
 	(segment
-		(start 163.4 85.4)
-		(end 162 84)
-		(width 1.25)
+		(start 167.78 73.43)
+		(end 167 72.65)
+		(width 1)
 		(layer "B.Cu")
 		(net 9)
 	)
 	(segment
-		(start 162 84)
-		(end 162 74)
-		(width 1.25)
-		(layer "B.Cu")
-		(net 9)
-	)
-	(segment
-		(start 159.7 68)
+		(start 159.65 67.95)
 		(end 155.95 64.25)
-		(width 1)
-		(layer "B.Cu")
-		(net 10)
-	)
-	(segment
-		(start 166 68)
-		(end 159.7 68)
 		(width 1)
 		(layer "B.Cu")
@@
 	)
 	(segment
+		(start 164.04 67.95)
+		(end 159.65 67.95)
+		(width 1)
+		(layer "B.Cu")
+		(net 10)
+	)
+	(segment
 		(start 149.05 50.2875)
 		(end 154.575 50.2875)
@@
 		(hatch edge 0.5)
 		(connect_pads
-			(clearance 0.5)
+			(clearance 1)
 		)
 		(min_thickness 0.25)

Commit message: update
Routing:
- net Net-(SW1-B): track 17.5 -> 18.9 mm
Changed lines of the file:
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@@
 	)
 	(segment
-		(start 167.78 81.61)
+		(start 166.35 85.35)
+		(end 167.78 83.92)
+		(width 1)
+		(layer "B.Cu")
+		(net 9)
+	)
+	(segment
+		(start 167.78 83.92)
 		(end 167.78 73.43)
+		(width 1)
+		(layer "B.Cu")
+		(net 9)
+	)
+	(segment
+		(start 167.78 73.43)
+		(end 167 72.65)
+		(width 1)
+		(layer "B.Cu")
+		(net 9)
+	)
+	(segment
+		(start 164.04 85.35)
+		(end 166.35 85.35)
 		(width 1)
 		(layer "B.Cu")
@@
 		(width 1)
 		(layer "B.Cu")
-		(net 9)
-	)
-	(segment
-		(start 164.04 85.35)
-		(end 167.78 81.61)
-		(width 1)
-		(layer "B.Cu")
-		(net 9)
-	)
-	(segment
-		(start 167.78 73.43)
-		(end 167 72.65)
-		(width 1)
-		(layer "B.Cu")

Commit message: actualizacion
Parts:
- removed the REF** at (167.8, 48.4)
- removed the REF** at (167.8, 102.7)
- removed the REF** at (123.8, 48.4)
- removed the REF** at (123.8, 102.7)
- added C3: 0.33uF, Capacitor_THT:CP_Radial_D5.0mm_P2.50mm, F.Cu at (96.0, 69.0)
- added G***: LOGO, RamLib:5i, B.Cu at (60.0, 50.0)
- added REF**: MountingHole_2.2mm_M2, MountingHole:MountingHole_2.2mm_M2, F.Cu at (49.0, 104.0)
- added REF**: MountingHole_2.2mm_M2, MountingHole:MountingHole_2.2mm_M2, F.Cu at (98.0, 104.0)
- added REF**: MountingHole_2.2mm_M2, MountingHole:MountingHole_2.2mm_M2, F.Cu at (49.0, 50.0)
- C1: footprint Capacitor_THT:CP_Radial_D5.0mm_P2.00mm -> Capacitor_THT:CP_Radial_D5.0mm_P2.50mm
- J1: value BTS7960_1 -> Screw_Terminal_01x08; footprint Connector_JST:JST_EH_B4B-EH-A_1x04_P2.50mm_Vertical -> Connector_IDC:IDC-Header_2x04_P2.54mm_Vertical
- J2: value BTS7960_2 -> Screw_Terminal_01x08; footprint Connector_JST:JST_EH_B4B-EH-A_1x04_P2.50mm_Vertical -> Connector_IDC:IDC-Header_2x04_P2.54mm_Vertical
- moved U1 75.0 mm to (61.3, 79.2)
- moved J2 73.6 mm to (81.5, 89.8), turned to 0 degrees
- moved J1 71.2 mm to (84.0, 77.0), turned to 180 degrees
- moved U2 70.2 mm to (93.5, 54.9), turned to 90 degrees
- moved C1 70.1 mm to (85.0, 59.0)
- moved SW1 69.2 mm to (95.4, 81.0)
- moved Logica_7.4v1 69.1 mm to (95.4, 95.5)
- moved C2 68.6 mm to (81.0, 58.0)
Connections:
- J1 pad 3: +5V -> unconnected-(J1-Pin_3-Pad3)
- J1 pad 4: GND -> unconnected-(J1-Pin_4-Pad4)
- J2 pad 1: GND -> LPWM_2
- J2 pad 2: +5V -> RPWM_2
- J2 pad 3: LPWM_2 -> unconnected-(J2-Pin_3-Pad3)
- J2 pad 4: RPWM_2 -> unconnected-(J2-Pin_4-Pad4)
- U1 pad 10: unconnected-(U1-IO27-Pad10) -> L_EN1
- U1 pad 11: unconnected-(U1-IO14-Pad11) -> L_EN2
Routing:
- net L_EN2: track 0.00 -> 52.8 mm
- net +5V: track 14.1 -> 65.5 mm
- net L_EN1: track 0.00 -> 12.0 mm
- net RPWM_2: track 6.61 -> 14.5 mm
- net LPWM_2: track 6.51 -> 10.4 mm
- net LPWM_1: track 10.0 -> 13.7 mm
- net Net-(SW1-B): track 18.9 -> 16.2 mm
- net RPWM_1: track 9.99 -> 9.28 mm
Other:
- board size 50 x 60 mm -> 55 x 60 mm

Commit message: actualizacion
Parts:
- moved C1 6.80 mm to (81.0, 53.5)
- moved C2 1.36 mm to (82.0, 57.0), turned to 0 degrees
- moved G*** 1.00 mm to (60.0, 51.0)
Connections:
- U1 pad 11: L_EN2 -> unconnected-(U1-IO14-Pad11)
- U1 pad 13: unconnected-(U1-IO13-Pad13) -> L_EN2
Routing:
- net L_EN2: track 52.8 -> 57.7 mm
- net Net-(SW1-B): track 16.2 -> 19.6 mm
- net +5V: track 65.5 -> 67.6 mm
- net L_EN1: track 12.0 -> 13.7 mm
- net unconnected-(U1-IO14-Pad11): track 0.00 -> 1.08 mm
Changed lines of the file:
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@@
 	(net 13 "unconnected-(U1-SD2-Pad14)")
 	(net 14 "unconnected-(U1-IO4-Pad26)")
-	(net 15 "unconnected-(U1-IO13-Pad13)")
+	(net 15 "unconnected-(U1-IO14-Pad11)")
 	(net 16 "unconnected-(U1-SD3-Pad15)")
 	(net 17 "unconnected-(U1-RX0-Pad33)")
@@
 	(footprint "Capacitor_THT:CP_Radial_D5.0mm_P2.50mm"
 		(layer "F.Cu")
-		(at 85 59 90)
+		(at 81 53.5 90)
 		(descr "CP, Radial series, Radial, pin pitch=2.50mm, , diameter=5mm, Electrolytic Capacitor")
 		(tags "CP Radial series Radial pin pitch 2.50mm  diameter 5mm Electrolytic Capacitor")
@@
 			(layers "*.Cu" "*.Mask" "F.SilkS")
 			(remove_unused_layers no)
-			(net 39 "L_EN2")
+			(net 15 "unconnected-(U1-IO14-Pad11)")
 			(pinfunction "IO14")
 			(pintype "bidirectional")
@@
 			(layers "*.Cu" "*.Mask" "F.SilkS")
 			(remove_unused_layers no)
-			(net 15 "unconnected-(U1-IO13-Pad13)")
+			(net 39 "L_EN2")
 			(pinfunction "IO13")
 			(pintype "bidirectional")
@@
 	(footprint "Capacitor_SMD:C_0805_2012Metric_Pad1.18x1.45mm_HandSolder"
 		(layer "B.Cu")
-		(at 81 57.9625 90)
+		(at 81.9625 57)
 		(descr "Capacitor SMD 0805 (2012 Metric), square (rectangular) end terminal, IPC_7351 nominal with elongated pad for handsoldering. (Body size source: IPC-SM-782 page 76, https://www.pcb-3d.com/wordpress/wp-content/uploads/ipc-sm-782a_amendment_1_and_2.pdf, https://docs.google.com/spreadsheets/d/1BsfQQcO9C6DZCsRaXUlFlo91Tg2WpOkGARC1WS5S8t0/edit?usp=sharing), generated with kicad-footprint-generator")
 		(tags "capacitor handsolder")
 		(property "Reference" "C2"
-			(at 0 1.68 90)
+			(at 0 1.68 0)
 			(layer "B.SilkS")
 			(effects
@@
 		)
 		(property "Value" "0.1uF"
-			(at 0 -1.68 90)
+			(at 0 -1.68 0)
 			(layer "B.Fab")
 			(effects
@@
 		)
 		(property "Datasheet" ""
-			(at 0 0 270)
+			(at 0 0 180)
 			(unlocked yes)
 			(layer "B.Fab")
@@
 		)
 		(property "Description" "Unpolarized capacitor"
-			(at 0 0 270)
+			(at 0 0 180)
 			(unlocked yes)
 			(layer "B.Fab")
@@
 		)
 		(fp_line
-			(start 1.88 -0.98)
-			(end -1.88 -0.98)
+			(start -1.88 -0.98)
+			(end -1.88 0.98)
 			(stroke
 				(width 0.05)
@@
 		)
 		(fp_line
-			(start -1.88 -0.98)
-			(end -1.88 0.98)
+			(start -1.88 0.98)
+			(end 1.88 0.98)
 			(stroke
 				(width 0.05)
@@
 		)
 		(fp_line
-			(start 1.88 0.98)
-			(end 1.88 -0.98)
+			(start 1.88 -0.98)
+			(end -1.88 -0.98)
 			(stroke
 				(width 0.05)
@@
 		)
 		(fp_line
-			(start -1.88 0.98)
-			(end 1.88 0.98)
+			(start 1.88 0.98)
+			(end 1.88 -0.98)
 			(stroke
 				(width 0.05)
@@
 		)
 		(fp_line
-			(start 1 -0.625)
-			(end -1 -0.625)
+			(start -1 -0.625)
+			(end -1 0.625)
 			(stroke
 				(width 0.1)
@@
 		)
 		(fp_line
-			(start -1 -0.625)
-			(end -1 0.625)
+			(start -1 0.625)
+			(end 1 0.625)
 			(stroke
 				(width 0.1)
@@
 		)
 		(fp_line
-			(start 1 0.625)
-			(end 1 -0.625)
+			(start 1 -0.625)
+			(end -1 -0.625)
 			(stroke
 				(width 0.1)
@@
 		)
 		(fp_line
-			(start -1 0.625)
-			(end 1 0.625)
+			(start 1 0.625)
+			(end 1 -0.625)
 			(stroke
 				(width 0.1)
@@
 		)
 		(fp_text user "${REFERENCE}"
-			(at 0 0 90)
+			(at 0 0 0)
 			(layer "B.Fab")
 			(effects
@@
 		)
 		(pad "1" smd roundrect
-			(at -1.0375 0 90)
+			(at -1.0375 0)
 			(size 1.175 1.45)
 			(layers "B.Cu" "B.Mask" "B.Paste")
@@
 		)
 		(pad "2" smd roundrect
-			(at 1.0375 0 90)
+			(at 1.0375 0)
 			(size 1.175 1.45)
 			(layers "B.Cu" "B.Mask" "B.Paste")
@@
 	(footprint "RamLib:5i"
 		(layer "B.Cu")
-		(at 60 50 180)
+		(at 60 51 180)
 		(property "Reference" "G***"
 			(at 0 0 0)
@@
 	)
 	(segment
-		(start 95.381 81)
-		(end 92 84.381)
+		(start 92 93)
+		(end 91 92)
 		(width 1)
 		(layer "B.Cu")
@@
 	)
 	(segment
-		(start 92 92)
-		(end 93 93)
+		(start 91 82)
+		(end 92 81)
 		(width 1)
 		(layer "B.Cu")
@@
 	)
 	(segment
-		(start 93 93)
-		(end 95.381 93)
+		(start 91 92)
+		(end 91 82)
 		(width 1)
 		(layer "B.Cu")
@@
 	)
 	(segment
-		(start 92 84.381)
-		(end 92 92)
+		(start 92 81)
+		(end 95.381 81)
+		(width 1)
+		(layer "B.Cu")
+		(net 9)
+	)
+	(segment
+		(start 95.381 93)
+		(end 92 93)
 		(width 1)
 		(layer "B.Cu")
@@
 	)
 	(segment
-		(start 87.087735 96.912265)
-		(end 86.54 97.46)
+		(start 74.01 74.17)
+		(end 73.17 74.17)
 		(width 1)
 		(layer "B.Cu")
-		(net 31)
+		(net 15)
 	)
 	(segment
-		(start 86 69.38)
-		(end 87.087735 70.467735)
+		(start 73.17 74.17)
+		(end 73 74)
+		(width 1)
+		(layer "B.Cu")
+		(net 15)
+	)
+	(segment
+		(start 87.087735 96.912265)
+		(end 86.54 97.46)
 		(width 1)
 		(layer "B.Cu")
@@
 	)
 	(segment
-		(start 84 67)
-		(end 84 69.38)
+		(start 86 69.38)
+		(end 87.087735 70.467735)
 		(width 1)
 		(layer "B.Cu")
@@
 	)
 	(segment
-		(start 86.5426 62.5426)
-		(end 90.92 62.5426)
+		(start 83.5 53.5)
+		(end 81 53.5)
 		(width 1)
 		(layer "B.Cu")
@@
 	)
 	(segment
-		(start 79.0635 59)
-		(end 81 59)
+		(start 86.54 97.46)
+		(end 84.02 97.46)
 		(width 1)
 		(layer "B.Cu")
@@
 	)
 	(segment
-		(start 74.01 56.39)
-		(end 76.4535 56.39)
+		(start 84 67)
+		(end 84 69.38)
 		(width 1)
 		(layer "B.Cu")
@@
 	)
 	(segment
-		(start 86.54 97.46)
-		(end 84.02 97.46)
+		(start 80.925 63.925)
+		(end 84 67)
 		(width 1)
 		(layer "B.Cu")
@@
 	(segment
 		(start 85 61)
-		(end 86.5426 62.5426)
+		(end 85 55)
 		(width 1)
 		(layer "B.Cu")
@@
 	)
 	(segment
-		(start 81 59)
-		(end 85 59)
+		(start 80.925 57)
+		(end 80.925 63.925)
 		(width 1)
 		(layer "B.Cu")
@@
 	)
 	(segment
-		(start 81 59)
-		(end 81 64)
+		(start 80.925 57)
+		(end 80.925 53.575)
 		(width 1)
 		(layer "B.Cu")
@@
 	)
 	(segment
-		(start 76.4535 56.39)
-		(end 79.0635 59)
+		(start 85 55)
+		(end 83.5 53.5)
 		(width 1)
 		(layer "B.Cu")
@@
 	)
 	(segment
-		(start 85 59)
+		(start 86.5426 62.5426)
 		(end 85 61)
 		(width 1)
@@
 	)
 	(segment
-		(start 81 64)
-		(end 84 67)
+		(start 90.92 62.5426)
+		(end 86.5426 62.5426)
 		(width 1)
 		(layer "B.Cu")
@@
 	)
 	(segment
-		(start 81.08 71.92)
-		(end 76.29 76.71)
+		(start 80.925 53.575)
+		(end 81 53.5)
+		(width 1)
+		(layer "B.Cu")
+		(net 31)
+	)
+	(segment
+		(start 76.29 76.71)
+		(end 77 76)
 		(width 1)
 		(layer "B.Cu")
@@
 	)
 	(segment
-		(start 81.46 71.92)
-		(end 81.08 71.92)
+		(start 74.01 76.71)
+		(end 76.29 76.71)
 		(width 1)
 		(layer "B.Cu")
@@
 	)
 	(segment
-		(start 84 71.92)
-		(end 81.46 71.92)
+		(start 77 73)
+		(end 78.08 71.92)
 		(width 1)
 		(layer "B.Cu")
@@
 	)
 	(segment
-		(start 76.29 76.71)
-		(end 74.01 76.71)
+		(start 78.08 71.92)
+		(end 81.46 71.92)
 		(width 1)
 		(layer "B.Cu")
@@
 	)
 	(segment
-		(start 74.01 74.17)
-		(end 73.17 74.17)
+		(start 77 76)
+		(end 77 73)
 		(width 1)
 		(layer "B.Cu")
-		(net 39)
+		(net 34)
 	)
 	(segment
-		(start 70 102)
-		(end 71 103)
+		(start 84 71.92)
+		(end 81.46 71.92)
 		(width 1)
 		(layer "B.Cu")
-		(net 39)
+		(net 34)
 	)
 	(segment
-		(start 73.17 74.17)
-		(end 73 74)
+		(start 78 96)
+		(end 78 102)
 		(width 1)
 		(layer "B.Cu")
@@
 	)
 	(segment
-		(start 71 74)
-		(end 70 75)
+		(start 79.08 94.92)
+		(end 78 96)
 		(width 1)
 		(layer "B.Cu")
@@
 	)
 	(segment
-		(start 71 103)
+		(start 78 102)
 		(end 77 103)
 		(width 1)
@@
 	)
 	(segment
-		(start 78 102)
-		(end 78 96)
+		(start 81.48 94.92)
+		(end 79.08 94.92)
 		(width 1)
 		(layer "B.Cu")
@@
 	)
 	(segment
-		(start 73 74)
-		(end 71 74)
+		(start 70 70)
+		(end 70.91 69.09)
 		(width 1)
 		(layer "B.Cu")
@@
 	)
 	(segment
-		(start 78 96)
-		(end 79.08 94.92)
+		(start 77 103)
+		(end 71 103)
 		(width 1)
 		(layer "B.Cu")
@@
 	)
 	(segment
-		(start 79.08 94.92)
-		(end 81.48 94.92)
+		(start 71 103)
+		(end 70 102)
 		(width 1)
 		(layer "B.Cu")
@@
 	)
 	(segment
-		(start 70 75)
-		(end 70 102)
+		(start 70.91 69.09)
+		(end 74.01 69.09)
 		(width 1)
 		(layer "B.Cu")
@@
 	)
 	(segment
-		(start 77 103)
-		(end 78 102)
+		(start 70 102)
+		(end 70 70)
 		(width 1)
 		(layer "B.Cu")
