File: Hardware/SumoRc/Sumorc.kicad_pcb (KiCad board)
At the start: 2 copper layers, 55 x 60 mm, 13 parts, among them J1 Screw_Terminal_01x08, J2 Screw_Terminal_01x08, SW1 SW_SPDT, U1 ESP32_DevKit_V1_DOIT, U2 LF15_TO220

Commit message: actualizacion
Parts:
- moved C2 0.61 mm to (82.0, 56.4)
Connections:
- J1 pad 3: unconnected-(J1-Pin_3-Pad3) -> +5V
- J1 pad 4: unconnected-(J1-Pin_4-Pad4) -> +5V
- J1 pad 5: L_EN1 -> unconnected-(J1-Pin_5-Pad5)
- J1 pad 6: L_EN1 -> unconnected-(J1-Pin_6-Pad6)
- J2 pad 3: unconnected-(J2-Pin_3-Pad3) -> +5V
- J2 pad 4: unconnected-(J2-Pin_4-Pad4) -> +5V
- J2 pad 5: L_EN2 -> unconnected-(J2-Pin_5-Pad5)
- J2 pad 6: L_EN2 -> unconnected-(J2-Pin_6-Pad6)
- J2 pad 7: GND -> +5V
- J2 pad 8: +5V -> GND
- U1 pad 10: L_EN1 -> R_EN1
- U1 pad 13: L_EN2 -> R_EN2
Routing:
- net L_EN2: track 57.7 -> 0.00 mm
- net +5V: track 67.6 -> 90.9 mm
- net L_EN1: track 13.7 -> 0.00 mm
- net unconnected-(U1-IO14-Pad11): track 1.08 -> 0.00 mm
Changed lines of the file:
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@@
 	(net 32 "unconnected-(U1-CLK-Pad20)")
 	(net 33 "unconnected-(U1-IO18-Pad30)")
-	(net 34 "L_EN1")
+	(net 34 "unconnected-(J1-Pin_5-Pad5)")
 	(net 35 "unconnected-(U1-IO2-Pad25)")
 	(net 36 "unconnected-(U1-EN-Pad1)")
 	(net 37 "unconnected-(U1-IO35-Pad5)")
 	(net 38 "unconnected-(U1-3V3-Pad19)")
-	(net 39 "L_EN2")
-	(net 40 "unconnected-(J1-Pin_4-Pad4)")
-	(net 41 "unconnected-(J1-Pin_3-Pad3)")
-	(net 42 "unconnected-(J2-Pin_3-Pad3)")
-	(net 43 "unconnected-(J2-Pin_4-Pad4)")
+	(net 39 "unconnected-(J1-Pin_6-Pad6)")
+	(net 40 "unconnected-(J2-Pin_5-Pad5)")
+	(net 41 "unconnected-(J2-Pin_6-Pad6)")
+	(net 42 "R_EN1")
+	(net 43 "R_EN2")
 	(footprint "Capacitor_THT:CP_Radial_D5.0mm_P2.50mm"
 		(layer "F.Cu")
@@
 		(pad "1" thru_hole rect
 			(at 0 0 90)
-			(size 1.6 1.6)
+			(size 1.9 1.9)
 			(drill 0.8)
 			(layers "*.Cu" "*.Mask")
@@
 		(pad "2" thru_hole circle
 			(at 2.5 0 90)
-			(size 1.6 1.6)
+			(size 2.3 2.3)
 			(drill 0.8)
 			(layers "*.Cu" "*.Mask")
@@
 			(layers "*.Cu" "*.Mask")
 			(remove_unused_layers no)
-			(net 42 "unconnected-(J2-Pin_3-Pad3)")
+			(net 31 "+5V")
 			(pinfunction "Pin_3")
 			(pintype "passive")
@@
 			(layers "*.Cu" "*.Mask")
 			(remove_unused_layers no)
-			(net 43 "unconnected-(J2-Pin_4-Pad4)")
+			(net 31 "+5V")
 			(pinfunction "Pin_4")
 			(pintype "passive")
@@
 			(layers "*.Cu" "*.Mask")
 			(remove_unused_layers no)
-			(net 39 "L_EN2")
+			(net 40 "unconnected-(J2-Pin_5-Pad5)")
 			(pinfunction "Pin_5")
-			(pintype "passive")
+			(pintype "passive+no_connect")
 		)
 		(pad "6" thru_hole oval
@@
 			(layers "*.Cu" "*.Mask")
 			(remove_unused_layers no)
-			(net 39 "L_EN2")
+			(net 41 "unconnected-(J2-Pin_6-Pad6)")
 			(pinfunction "Pin_6")
-			(pintype "passive")
+			(pintype "passive+no_connect")
 		)
 		(pad "7" thru_hole oval
@@
 			(layers "*.Cu" "*.Mask")
 			(remove_unused_layers no)
-			(net 1 "GND")
+			(net 31 "+5V")
 			(pinfunction "Pin_7")
 			(pintype "passive")
@@
 			(layers "*.Cu" "*.Mask")
 			(remove_unused_layers no)
-			(net 31 "+5V")
+			(net 1 "GND")
 			(pinfunction "Pin_8")
 			(pintype "passive")
@@
 		(pad "1" thru_hole rect
 			(at 0 0 180)
-			(size 1.6 1.6)
+			(size 1.9 1.9)
 			(drill 0.8)
 			(layers "*.Cu" "*.Mask")
@@
 		(pad "2" thru_hole circle
 			(at 2.5 0 180)
-			(size 1.6 1.6)
+			(size 2.3 2.3)
 			(drill 0.8)
 			(layers "*.Cu" "*.Mask")
@@
 			(layers "*.Cu" "*.Mask" "F.SilkS")
 			(remove_unused_layers no)
-			(net 34 "L_EN1")
+			(net 42 "R_EN1")
 			(pinfunction "IO27")
 			(pintype "bidirectional")
@@
 			(layers "*.Cu" "*.Mask" "F.SilkS")
 			(remove_unused_layers no)
-			(net 39 "L_EN2")
+			(net 43 "R_EN2")
 			(pinfunction "IO13")
 			(pintype "bidirectional")
@@
 			(layers "*.Cu" "*.Mask")
 			(remove_unused_layers no)
-			(net 41 "unconnected-(J1-Pin_3-Pad3)")
+			(net 31 "+5V")
 			(pinfunction "Pin_3")
 			(pintype "passive")
@@
 			(layers "*.Cu" "*.Mask")
 			(remove_unused_layers no)
-			(net 40 "unconnected-(J1-Pin_4-Pad4)")
+			(net 31 "+5V")
 			(pinfunction "Pin_4")
 			(pintype "passive")
@@
 			(layers "*.Cu" "*.Mask")
 			(remove_unused_layers no)
-			(net 34 "L_EN1")
+			(net 34 "unconnected-(J1-Pin_5-Pad5)")
 			(pinfunction "Pin_5")
-			(pintype "passive")
+			(pintype "passive+no_connect")
 		)
 		(pad "6" thru_hole oval
@@
 			(layers "*.Cu" "*.Mask")
 			(remove_unused_layers no)
-			(net 34 "L_EN1")
+			(net 39 "unconnected-(J1-Pin_6-Pad6)")
 			(pinfunction "Pin_6")
-			(pintype "passive")
+			(pintype "passive+no_connect")
 		)
 		(pad "7" thru_hole oval
@@
 	(footprint "Capacitor_SMD:C_0805_2012Metric_Pad1.18x1.45mm_HandSolder"
 		(layer "B.Cu")
-		(at 81.9625 57)
+		(at 82.0375 56.39)
 		(descr "Capacitor SMD 0805 (2012 Metric), square (rectangular) end terminal, IPC_7351 nominal with elongated pad for handsoldering. (Body size source: IPC-SM-782 page 76, https://www.pcb-3d.com/wordpress/wp-content/uploads/ipc-sm-782a_amendment_1_and_2.pdf, https://docs.google.com/spreadsheets/d/1BsfQQcO9C6DZCsRaXUlFlo91Tg2WpOkGARC1WS5S8t0/edit?usp=sharing), generated with kicad-footprint-generator")
 		(tags "capacitor handsolder")
@@
 	)
 	(segment
-		(start 74.01 74.17)
-		(end 73.17 74.17)
+		(start 81 63.85)
+		(end 81 58)
 		(width 1)
 		(layer "B.Cu")
-		(net 15)
+		(net 31)
 	)
 	(segment
-		(start 73.17 74.17)
-		(end 73 74)
+		(start 86 69.38)
+		(end 87.087735 70.467735)
 		(width 1)
 		(layer "B.Cu")
-		(net 15)
+		(net 31)
 	)
 	(segment
-		(start 87.087735 96.912265)
-		(end 86.54 97.46)
+		(start 84 69.38)
+		(end 86 69.38)
 		(width 1)
 		(layer "B.Cu")
@@
 	)
 	(segment
-		(start 86 69.38)
-		(end 87.087735 70.467735)
+		(start 84.02 92.38)
+		(end 85.707735 92.38)
 		(width 1)
 		(layer "B.Cu")
@@
 	)
 	(segment
-		(start 84 69.38)
-		(end 86 69.38)
+		(start 86 61)
+		(end 86 55)
 		(width 1)
 		(layer "B.Cu")
@@
 	)
 	(segment
-		(start 83.5 53.5)
-		(end 81 53.5)
+		(start 86 55)
+		(end 84.5 53.5)
 		(width 1)
 		(layer "B.Cu")
@@
 	)
 	(segment
-		(start 86.54 97.46)
-		(end 84.02 97.46)
+		(start 84.02 92.38)
+		(end 81.48 92.38)
 		(width 1)
 		(layer "B.Cu")
@@
 	)
 	(segment
-		(start 84 67)
-		(end 84 69.38)
+		(start 85.707735 92.38)
+		(end 87.087735 91)
 		(width 1)
 		(layer "B.Cu")
@@
 	)
 	(segment
-		(start 80.925 63.925)
-		(end 84 67)
+		(start 84 74.46)
+		(end 85.627735 74.46)
+		(width 1)
+		(layer "B.Cu")
+		(net 31)
+	)
+	(segment
+		(start 81.46 74.46)
+		(end 84 74.46)
 		(width 1)
 		(layer "B.Cu")
@@
 	)
 	(segment
-		(start 85 61)
-		(end 85 55)
+		(start 81 56.39)
+		(end 80 56.39)
 		(width 1)
 		(layer "B.Cu")
@@
 	)
 	(segment
-		(start 80.925 57)
-		(end 80.925 63.925)
+		(start 79 93)
+		(end 79 96.5)
 		(width 1)
 		(layer "B.Cu")
@@
 	)
 	(segment
-		(start 80.925 57)
-		(end 80.925 53.575)
+		(start 80.925 63.925)
+		(end 81 63.85)
 		(width 1)
 		(layer "B.Cu")
@@
 	)
 	(segment
-		(start 85 55)
-		(end 83.5 53.5)
+		(start 79 96.5)
+		(end 79.96 97.46)
 		(width 1)
 		(layer "B.Cu")
@@
 	)
 	(segment
-		(start 86.5426 62.5426)
-		(end 85 61)
+		(start 81 55)
+		(end 81 55.39)
 		(width 1)
 		(layer "B.Cu")
@@
 	(segment
 		(start 90.92 62.5426)
-		(end 86.5426 62.5426)
+		(end 87.5426 62.5426)
 		(width 1)
 		(layer "B.Cu")
@@
 	)
 	(segment
-		(start 87.087735 70.467735)
-		(end 87.087735 96.912265)
+		(start 79.62 92.38)
+		(end 79 93)
 		(width 1)
 		(layer "B.Cu")
@@
 	)
 	(segment
-		(start 80.925 53.575)
-		(end 81 53.5)
+		(start 81.48 92.38)
+		(end 79.62 92.38)
 		(width 1)
 		(layer "B.Cu")
@@
 	)
 	(segment
-		(start 76.29 76.71)
-		(end 77 76)
+		(start 81 57.39)
+		(end 80 56.39)
 		(width 1)
 		(layer "B.Cu")
-		(net 34)
+		(net 31)
 	)
 	(segment
-		(start 74.01 76.71)
-		(end 76.29 76.71)
+		(start 80.925 63.925)
+		(end 84 67)
 		(width 1)
 		(layer "B.Cu")
-		(net 34)
+		(net 31)
 	)
 	(segment
-		(start 77 73)
-		(end 78.08 71.92)
+		(start 87.087735 73)
+		(end 87.087735 91)
 		(width 1)
 		(layer "B.Cu")
-		(net 34)
+		(net 31)
 	)
 	(segment
-		(start 78.08 71.92)
-		(end 81.46 71.92)
+		(start 81 53.5)
+		(end 81 55)
 		(width 1)
 		(layer "B.Cu")
-		(net 34)
+		(net 31)
 	)
 	(segment
-		(start 77 76)
-		(end 77 73)
+		(start 80 56.39)
+		(end 74.01 56.39)
 		(width 1)
 		(layer "B.Cu")
-		(net 34)
+		(net 31)
 	)
 	(segment
-		(start 84 71.92)
-		(end 81.46 71.92)
+		(start 87.5426 62.5426)
+		(end 86 61)
 		(width 1)
 		(layer "B.Cu")
-		(net 34)
+		(net 31)
 	)
 	(segment
-		(start 78 96)
-		(end 78 102)
+		(start 81 58)
+		(end 81 56.39)
 		(width 1)
 		(layer "B.Cu")
-		(net 39)
+		(net 31)
 	)
 	(segment
-		(start 84.02 94.92)
-		(end 81.48 94.92)
+		(start 81 55)
+		(end 81 56.39)
 		(width 1)
 		(layer "B.Cu")
-		(net 39)
+		(net 31)
 	)
 	(segment
-		(start 79.08 94.92)
-		(end 78 96)
+		(start 81 58)
+		(end 81 57.39)
 		(width 1)
 		(layer "B.Cu")
-		(net 39)
+		(net 31)
 	)
 	(segment
-		(start 78 102)
-		(end 77 103)
+		(start 81 55.39)
+		(end 80 56.39)
 		(width 1)
 		(layer "B.Cu")
-		(net 39)
+		(net 31)
 	)
 	(segment
-		(start 81.48 94.92)
-		(end 79.08 94.92)
+		(start 79.96 97.46)
+		(end 81.48 97.46)
 		(width 1)
 		(layer "B.Cu")
-		(net 39)
+		(net 31)
 	)
 	(segment
-		(start 70 70)
-		(end 70.91 69.09)
+		(start 87.087735 70.467735)
+		(end 87.087735 73)
 		(width 1)
 		(layer "B.Cu")
-		(net 39)
+		(net 31)
 	)
 	(segment
-		(start 77 103)
-		(end 71 103)
+		(start 80.925 53.575)
+		(end 81 53.5)
 		(width 1)
 		(layer "B.Cu")
-		(net 39)
+		(net 31)
 	)
 	(segment
-		(start 71 103)
-		(end 70 102)
+		(start 84.5 53.5)
+		(end 81 53.5)
 		(width 1)
 		(layer "B.Cu")
-		(net 39)
+		(net 31)
 	)
 	(segment
-		(start 70.91 69.09)
-		(end 74.01 69.09)
+		(start 84 67)
+		(end 84 69.38)
 		(width 1)
 		(layer "B.Cu")
-		(net 39)
+		(net 31)
 	)
 	(segment
-		(start 70 102)
-		(end 70 70)
+		(start 85.627735 74.46)
+		(end 87.087735 73)
 		(width 1)
 		(layer "B.Cu")
-		(net 39)
+		(net 31)
 	)
 	(zone
